Commit message: update

File: resources/robots/bhr8fc2/bhr8fc2mc_add_pos_limit.urdf (robot description, URDF)
Before this commit: robot bhr8_fc2, 21 links, 20 joints
Joints:
- joint lankle1: limit lower=-3.14 upper=3.14 effort=100.0 velocity=100.0 -> lower=-1.0 upper=0.6 effort=300.0 velocity=21.0
- joint lankle2: limit lower=-3.14 upper=3.14 effort=100.0 velocity=100.0 -> lower=-0.78 upper=0.78 effort=300.0 velocity=21.0
- joint lelbow: limit lower=-3.14 upper=3.14 effort=100.0 velocity=100.0 -> lower=0.0 upper=2.0 effort=300 velocity=21.0
- joint lhipPitch: limit lower=-3.14 upper=3.14 effort=100.0 velocity=100.0 -> lower=-1.4 upper=0.7 effort=300.0 velocity=21.0
- joint lhipRoll: limit lower=-3.14 upper=3.14 effort=100.0 velocity=100.0 -> lower=-0.78 upper=0.78 effort=300.0 velocity=21.0
- joint lhipYaw: limit lower=-3.14 upper=3.14 effort=100.0 velocity=100.0 -> lower=-0.78 upper=0.78 effort=300.0 velocity=21.0
- joint lknee: limit lower=-3.14 upper=3.14 effort=100.0 velocity=100.0 -> lower=0 upper=1.8 effort=300.0 velocity=21.0
- joint lshoulderPitch: limit lower=-3.14 upper=3.14 effort=100.0 velocity=100.0 -> lower=-3.14 upper=3.14 effort=300 velocity=21.0
- joint lshoulderRoll: limit lower=-3.14 upper=3.14 effort=100.0 velocity=100.0 -> lower=0 upper=1.57 effort=300 velocity=21.0
- joint lshoulderYaw: limit lower=-3.14 upper=3.14 effort=100.0 velocity=100.0 -> lower=-1.57 upper=1.57 effort=300 velocity=21.0
- joint rankle1: limit lower=-3.14 upper=3.14 effort=100.0 velocity=100.0 -> lower=-1.0 upper=0.6 effort=300.0 velocity=21.0
- joint rankle2: limit lower=-3.14 upper=3.14 effort=100.0 velocity=100.0 -> lower=-0.78 upper=0.78 effort=300.0 velocity=21
- joint relbow: limit lower=-3.14 upper=3.14 effort=100.0 velocity=100.0 -> lower=0.0 upper=2.0 effort=300 velocity=21.0
- joint rhipPitch: limit lower=-3.14 upper=3.14 effort=100.0 velocity=100.0 -> lower=-1.4 upper=0.7 effort=300.0 velocity=21.0
- joint rhipRoll: limit lower=-3.14 upper=3.14 effort=100.0 velocity=100.0 -> lower=-0.78 upper=0.78 effort=300.0 velocity=21.0
- joint rhipYaw: limit lower=-3.14 upper=3.14 effort=100.0 velocity=100.0 -> lower=-0.78 upper=0.78 effort=300.0 velocity=21.0
- joint rknee: limit lower=-3.14 upper=3.14 effort=100.0 velocity=100.0 -> lower=0 upper=1.8 effort=300.0 velocity=21.0
- joint rshoulderPitch: limit lower=-3.14 upper=3.14 effort=100.0 velocity=100.0 -> lower=-3.14 upper=3.14 effort=300.0 velocity=21.0
- joint rshoulderRoll: limit lower=-3.14 upper=3.14 effort=100.0 velocity=100.0 -> lower=-1.57 upper=0 effort=300 velocity=21.0
- joint rshoulderYaw: limit lower=-3.14 upper=3.14 effort=100.0 velocity=100.0 -> lower=-1.57 upper=1.57 effort=300 velocity=21.0
